File: projects/cckb/pcb/cckb_main.kicad_pcb (KiCad board)
At the start: 2 copper layers, 286.4 x 95.9 mm, 145 parts, among them SW1 PG1350, SW10 PG1350, SW11 PG1350, SW12 PG1350, SW13 PG1350, SW14 PG1350, SW15 PG1350, SW16 PG1350, SW17 PG1350, SW18 PG1350, SW19 PG1350, SW2 PG1350, SW20 PG1350, SW21 PG1350, SW22 PG1350, SW23 PG1350, SW24 PG1350, SW25 PG1350, SW26 PG1350, SW27 PG1350, SW28 PG1350, SW29 PG1350, SW3 PG1350, SW30 PG1350, SW31 PG1350, SW32 PG1350, SW33 PG1350, SW34 PG1350, SW35 PG1350, SW36 PG1350, SW37 PG1350, SW38 PG1350, SW39 PG1350, SW4 PG1350, SW40 PG1350, SW41 PG1350, SW42 PG1350, SW43 PG1350, SW44 PG1350, SW45 PG1350, SW46 PG1350, SW47 PG1350, SW48 PG1350, SW49 PG1350, SW5 PG1350, SW50 PG1350, SW51 PG1350, SW52 PG1350, SW53 PG1350, SW54 PG1350, SW55 PG1350, SW56 PG1350, SW57 PG1350, SW58 PG1350, SW59 PG1350, SW6 PG1350, SW60 PG1350, SW61 PG1350, SW62 PG1350, SW7 PG1350, SW8 PG1350, SW9 PG1350, U1 SN74LVC595APWR, U2 SN74LVC595APWR

Commit message: CCKB 監査の直し（R1〜R6）: パッドの中のビアを根本から無くし、XIAO の裏の露出パッド 8 個と H3 のインサートの下の表の銅を 0 に、電源スイッチを手はんだに、トレイの隙を片側 0.5 に
- R1: route_pcb.Space.free() が同じネットのパッドを当てていなかった（C_U1・BT1 の GND パッドの中に縫いのビア）。全パッドの「ビアが掛からない」検査（XIAO の D0〜D6 だけ名指しで例外）
- R2: SW_PWR を NOT_ASSEMBLED に（BOM 5 行・CPL 69 行）。Fabrication Toolkit の CPL を EasyEDA の原点とパッドで置き直して板と比べる検査
- R3: 露出パッド 8 個を STEP と Seeed 公式フットプリントで確定（spec.XIAO_BOTTOM_PADS）。XIAO のパッドを縁から内 2.2 に、禁止域を 8 個＋0.3 に
- R6: H3 のまわりに表の禁止域（半径 1.9）
- R5: spec.CASE_PCB_GAP 0.5 を interface が 1 か所で読む。外面は動かさず壁 1.3・窪み 0.9
- R7: パッド内ビア φ0.7・0805 と手はんだの GND をサーマル・ビア 1 本の長い GND の島に 2 本目
- 指紋がパッドの形とルール領域を見ない穴を、項目の比較と unrouted_sha256 で塞いだ

Co-Authored-By: Claude Opus 5.5 (1M context) <noreply@anthropic.com>
Routing:
- net CS: track 229.7 -> 399.5 mm, vias 1 -> 2
- net SPI_SCK: track 225.5 -> 236.4 mm
- net U1_U2: track 163.6 -> 157.8 mm, vias 2 -> 4
- net COL6: track 183.5 -> 179.2 mm
- net COL10: track 140.5 -> 143.7 mm
- net COL8: track 180.7 -> 178.8 mm
- net V3V3: track 242.8 -> 244.6 mm
- net COL3: track 131.6 -> 130.4 mm
- net COL5: track 161.0 -> 162.2 mm
- net COL0: track 128.3 -> 127.2 mm
- net COL4: track 114.1 -> 113.0 mm
- net COL2: track 98.4 -> 99.4 mm, vias 2 -> 0
- net COL12: track 122.9 -> 123.9 mm
- net VBAT_SW: track 289.3 -> 288.3 mm
- net COL7: track 168.5 -> 169.1 mm
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
Commit message: CCKB 2 回目の監査の直し（S1〜S3）: 金属が当たる 10 か所に禁止域、CS の 1 本だけ置き直し、D_PWR の既定を BAT46W に
- S1: interface.metal_on_pcb が取付の穴 11 ごとに金属の当たる面を高さで判定（上面にナット 9・H3 のインサート、下面 0）。
  METAL_KEEPOUT を 10 か所に。route_pcb.py --reroute CS で前の板の配線を持ってきて、H5・H6 のナットの下の CS の 1 本だけを
  決まった形で置き直した（ほかの 89 網は線・ビアとも前の板と同じ）。検査は板から穴を数え、塗った後の銅まで見る
- S2: 逆流を「逆漏れ − 分圧が吸う電流」・Vf を保証値どうしで比べ直し、既定を BAT46W C54110 に（利用者が発注前に決める・O12）
- S3: 手はんだの部品のパッドからペーストを外した（B_Paste 173 → 166）・パッド内ビア φ0.8・DRC の警告の数を固定・
  USB のシールドの長穴 4 個を数えに・つまみ 1.55×1.1・手順書と台帳

Co-Authored-By: Claude Opus 5.5 (1M context) <noreply@anthropic.com>
Parts:
- D_PWR: value B5819W -> BAT46W
Routing:
- net CS: track 399.5 -> 400.6 mm
- net GND: vias 999 -> 1003

Commit message: CCKB 電源スイッチを秋月 SS-12D00G3（表・レバーが上）へ: 基板・ケース・組み立て・検査
- 利用者の決定（2026-09-24）で MK-12C02-G025（LCSC・裏・横のつまみ）から置き換え
- 基板: SW_PWR を表・スルーホールで (141.225, -38.6)、BT1 を左へ 3.8（124.7）。
  網 VBAT_IN・VBAT_SW の右の角だけ引き直し（ほかの 88 網は前の板と同じ）。
  枠の爪の下に表の銅の禁止域 PSW_TAB_KEEPOUT。位置決めの穴が無くなり DRC_SEVERITY を消した
  （DRC 違反 0・未配線 0・警告 3）。前のフットプリントと EasyEDA の C778186 を消した
- route_pcb: --clear（動かした部品の周りの前の線を捨てる）・行き止まりの削除・
  SES の取り込みで動いた部品を元に戻す（A10 の 50nm の原因）・引き直す網を二重に戻さない
- ケース: 右の壁の切り欠き・窪み・ふたのひれを消し、右のふたにレバーの穴 6.4x2.4 と「ON ↑」の刻印
- 組み立て: スイッチを 1 つの立体に（足は 1.0 に切る）。爪の検査を上からに書き直し
- 爪の出 PSW_TAB 0.4 [暫定]（図面に寸法無し）でレバーの先は名目でふたの上面の 0.1 下・最悪 +0.2（O13）

Co-Authored-By: Claude Opus 5.5 (1M context) <noreply@anthropic.com>
Parts:
- removed the SW_PWR at (291.3, 143.4)
- added SW_PWR: SS-12D00G3, SW_SS-12D00G3, F.Cu at (291.2, 138.6)
- moved BT1 3.80 mm to (274.7, 138.6)
Routing:
- net VBAT_SW: track 288.3 -> 286.3 mm
- net VBAT_IN: track 6.16 -> 4.40 mm, vias 1 -> 0
- net GND: vias 1003 -> 1001

Commit message: CCKB を Choc V2 に: 基板を作り直して配線（DRC 違反 0・未配線 0）・高さ・床の止まり穴の出力
- spec: SWITCH=choc_v2・高さ 5.3/8.6・足の公差 0.2・中心の突起 3.30・床の止まり穴 0.4（UNDER_PCB 1.8 のまま）
- 行のバスを 3.35 下に（中心穴と位置決めの長穴の間）。スタビ・取付の穴の所だけ下へ回り道（matrix_routes.buses）
- 列が段の境目を渡る高さをずらせるように・XIAO から行 0〜2 は XIAO の下で左へ寄せてから上がる
- VBAT_SW の長い 1 本を決まった形で（POWER_RUNS）・D_PWR を XIAO の奥の縁の上へ
- 595 の OE を本体の下で GND の 8 番へ（ビア 1 本の OE が線に囲まれて浮いた）
- 長円の非めっき穴の縁に配線禁止の帯（NPTH_KEEPOUT）・縫いのビアは穴の実物の形で当てる
- 取付 H9 を Del の右下へ・H0 を 0.25 左へ・支え 8 本を動かした（当たり: 長穴・スタビの穴）
- interface.floor_pockets（突起 62・スタビの箱 8）をケースの段の出どころに
- 検査を V2 の値に。足の先と床の間が最悪 0.04 で高さ・剛性の検査 2 つは赤のまま（利用者の判断待ち）

Co-Authored-By: Claude Opus 5.5 (1M context) <noreply@anthropic.com>
Parts:
- added ST42: Stab_Kailh_Choc_V2_Screw_2u, Stab_Kailh_Choc_V2_Screw_2u, F.Cu at (271.4, 100.0)
- added ST43: Stab_Kailh_Choc_V2_Screw_2u, Stab_Kailh_Choc_V2_Screw_2u, F.Cu at (28.6, 119.0)
- added ST58: Stab_Kailh_Choc_V2_Screw_2u, Stab_Kailh_Choc_V2_Screw_2u, F.Cu at (104.8, 138.1)
- added ST60: Stab_Kailh_Choc_V2_Screw_2u, Stab_Kailh_Choc_V2_Screw_2u, F.Cu at (176.2, 138.1)
- SW1, SW10, SW11, SW12, SW13, SW14, SW15, SW16, SW17, SW18, SW19, SW2, SW20, SW21, SW22, SW23, SW24, SW25, SW26, SW27, SW28, SW29, SW3, SW30, SW31, SW32, SW33, SW34, SW35, SW36, SW37, SW38, SW39, SW4, SW40, SW41, SW42, SW43, SW44, SW45, SW46, SW47, SW48, SW49, SW5, SW50, SW51, SW52, SW53, SW54, SW55, SW56, SW57, SW58, SW59, SW6, SW60, SW61, SW62, SW7, SW8, SW9: value PG1350 -> PG1353; footprint SW_Kailh_Choc_V1 -> SW_Kailh_Choc_V2_Slot
- moved H9 21.9 mm to (289.4, 85.0)
- moved D42 4.20 mm to (278.5, 99.0), turned to 90 degrees
- moved D58 4.20 mm to (111.9, 137.1), turned to 90 degrees
- moved D43 4.20 mm to (35.7, 118.0), turned to 90 degrees
- moved D60 4.20 mm to (183.3, 137.1), turned to 90 degrees
- moved D_PWR 2.83 mm to (26.0, 128.4)
- moved D1 0.50 mm to (23.7, 60.9)
- moved D10 0.50 mm to (195.2, 60.9)
- moved D11 0.50 mm to (214.2, 60.9)
- moved D12 0.50 mm to (233.3, 60.9)
- moved D13 0.50 mm to (252.3, 60.9)
- moved D14 0.50 mm to (271.4, 60.9)
- moved D15 0.50 mm to (290.4, 60.9)
- moved D16 0.50 mm to (28.5, 79.9)
- moved D17 0.50 mm to (52.3, 79.9)
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Routing:
- net CS: track 400.6 -> 263.5 mm
- net ROW4: track 247.7 -> 288.4 mm
- net COL1: track 237.5 -> 255.7 mm, vias 1 -> 2
- net GND: track 16.8 -> 34.4 mm, vias 1001 -> 910
- net VBAT_SW: track 286.3 -> 301.3 mm
- net ROW0: track 426.3 -> 412.5 mm
- net ROW1: track 400.2 -> 387.4 mm
- net COL9: track 135.5 -> 145.7 mm
- net SPI_SCK: track 236.4 -> 226.8 mm, vias 1 -> 2
- net COL0: track 127.2 -> 136.0 mm
- net COL14: track 156.6 -> 163.4 mm
- net COL13: track 133.8 -> 140.1 mm
- net COL10: track 143.7 -> 149.4 mm
- net SW42_D: track 8.90 -> 3.25 mm
- net SW60_D: track 8.90 -> 3.25 mm
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Other:
- outline, holes or cut-outs redrawn

Commit message: CCKB V2 の位置決めの穴を丸 φ2.1 に（JLC の長円の比）・名札・床の穴: 板 6b886491（DRC 違反 0・未配線 0・警告 0）
2026-09-26 の V2 監査 C 重要 1: 非めっきの長円 78 個が JLC の「長円の長さ ≧ 幅 × 2」を満たさない。
- 位置決めの長円 62（1.6 × 2.0・比 1.25）を丸 φ2.1 に。足跡を SW_Kailh_Choc_V2_Slot → SW_Kailh_Choc_V2_Common。
  3 枚の図の推奨の穴（標準 φ1.60・静音 長円 2.0 × 1.5）の和を JLC の丸穴の公差 −0.08 でも含む。底面図の「5.50」は
  穴の中の突起と読み直した（静音 茶の図を 600dpi で）。突起は公差の最悪でも入る
- スタビのねじ・爪の長円 16 は保留（スタビの品を選び直し中。Kailh 公式 CPG1353G24D01）。検査は数を固定した例外 16
- 検査: 板の穴の比（board_facts に drill_wh・slot）と、発注の道具が出した NPTH.drl の長円。前の板で落ちることを確かめた
- 配線は前の板（dae52e33）の信号線を route_pcb --reroute でそのまま持ってきた（全部を引き直すと COL5・COL6 が未配線）。
  route_pcb は計画が引く網（ROW*・SW*_D）を前の板から持ってこない・長円が無いとき NPTH_KEEPOUT を求めない
- C 軽微 3: D42・D43・D58・D60 の名札をダイオードの左へ（silk_edge_clearance 4 → 0）
- 床の止まり穴（位置決め）が丸 φ2.9 に → 支えの柱 4 本を 0.1・左奥の滑り止めを 0.2 動かした
- E 重要 4: 枠がスイッチを保持しないことを mech のコメントに

Co-Authored-By: Claude Opus 5.5 (1M context) <noreply@anthropic.com>
Parts:
- SW1, SW10, SW11, SW12, SW13, SW14, SW15, SW16, SW17, SW18, SW19, SW2, SW20, SW21, SW22, SW23, SW24, SW25, SW26, SW27, SW28, SW29, SW3, SW30, SW31, SW32, SW33, SW34, SW35, SW36, SW37, SW38, SW39, SW4, SW40, SW41, SW42, SW43, SW44, SW45, SW46, SW47, SW48, SW49, SW5, SW50, SW51, SW52, SW53, SW54, SW55, SW56, SW57, SW58, SW59, SW6, SW60, SW61, SW62, SW7, SW8, SW9: footprint SW_Kailh_Choc_V2_Slot -> SW_Kailh_Choc_V2_Common
