File: projects/cckb/pcb/cckb_main.kicad_pcb (KiCad board)
At the start: 2 copper layers, 286.4 x 95.9 mm, 149 parts, among them SW1 PG1353, SW10 PG1353, SW11 PG1353, SW12 PG1353, SW13 PG1353, SW14 PG1353, SW15 PG1353, SW16 PG1353, SW17 PG1353, SW18 PG1353, SW19 PG1353, SW2 PG1353, SW20 PG1353, SW21 PG1353, SW22 PG1353, SW23 PG1353, SW24 PG1353, SW25 PG1353, SW26 PG1353, SW27 PG1353, SW28 PG1353, SW29 PG1353, SW3 PG1353, SW30 PG1353, SW31 PG1353, SW32 PG1353, SW33 PG1353, SW34 PG1353, SW35 PG1353, SW36 PG1353, SW37 PG1353, SW38 PG1353, SW39 PG1353, SW4 PG1353, SW40 PG1353, SW41 PG1353, SW42 PG1353, SW43 PG1353, SW44 PG1353, SW45 PG1353, SW46 PG1353, SW47 PG1353, SW48 PG1353, SW49 PG1353, SW5 PG1353, SW50 PG1353, SW51 PG1353, SW52 PG1353, SW53 PG1353, SW54 PG1353, SW55 PG1353, SW56 PG1353, SW57 PG1353, SW58 PG1353, SW59 PG1353, SW6 PG1353, SW60 PG1353, SW61 PG1353, SW62 PG1353, SW7 PG1353, SW8 PG1353, SW9 PG1353, U1 SN74LVC595APWR, U2 SN74LVC595APWR

Commit message: CCKB V2 スタビの穴を販売者の実測に（支点 ±11.9・丸 φ3.0 / φ4.0・半径 2.6 の禁止域）・プレート・キャップの受け口: 板 5f02d2b0（DRC 違反 0・未配線 0・警告 0）
- 基板: ねじ φ3.0 を y −6.2・爪 φ4.0 を y +8.24（丸い非めっき）・箱の穴 支点 ±3.0 × ±4.0。穴の中心から 2.6 は GND のベタ以外の銅なし（STAB_HOLE_KEEPOUT）
- 長円の例外 HELD_STAB_SLOTS を消した（板・ドリルのファイルとも長円 0）。発注する板を決めた数と比べる検査と壊す検査 7 通り
- 配線: 行のバスは禁止域の下を回る（キー中心の 8.95 下）。左 Shift の左のねじの禁止域で塞がった VBAT_SW・V3V3・SPI_MOSI と、行 2 の回り道に重なった COL14 を決まった形で（spec.FIXED_RUNS）
- プレート: 販売者の足跡の値に戻した（+0.1 を消した）。残した妥協 4 つ
- キャップ: 受け口を ±11.9・台 φ5.1 で 2.0 掴む（前 0.45）。coupon_stab_return。ねじの頭 φ3.7 × 1.5 と床の止まり穴 8・支え 2 本を動かした

Co-Authored-By: Claude Opus 5.5 (1M context) <noreply@anthropic.com>
Routing:
- net VBAT_SW: track 301.3 -> 321.2 mm
- net ROW4: track 288.4 -> 293.2 mm
- net ROW2: track 369.8 -> 371.0 mm
- net ROW3: track 338.9 -> 340.1 mm
- net V3V3: track 243.2 -> 243.3 mm, vias 2 -> 3
- net GND: vias 910 -> 893
Other:
- outline, holes or cut-outs redrawn

Commit message: CCKB V2 2 回目の監査の基板の直し: GND の縫いのビア 6・R_LO の名札・スタビの裏のコートヤード・穴と銅 0.28: 板 abcd20ff（DRC 違反 0・未配線 0・警告 0）
- D-1: 裏の GND の帯（ROW4 と手前の縁の間）に 5 本。帯の先から最寄りの GND のビアまで銅の上の道のり 33.3 → 3.1
- D-2: 表の島（左 Shift の左の箱の穴を VBAT_SW が U 字に囲む所）に 1 本。12.3 → 10.3。
  監査の勧めた左上は U の腕の幅 1.006 / 0.8 でビアが入らない（3 以下はビアでは届かない）
- 宣言した GND のビア spec.GND_STITCH_AT を route_pcb が最後に打つ（置けなければ止まる）。
  route_pcb --keep（何も引き直さず GND だけ作り直す）。変更前の板で --keep が線・ビア・塗りを同じに戻すことを確かめた
- C-3: R_LO の名札 3.2 → 3.35（マスクの開口まで 0.081 → 0.231）
- C-4: .kicad_pro の min_hole_clearance 0.28（spec.DRC_PTH_HOLE_CLEARANCE・pcb_rules.JLC["pth_to_track"]）。
  前の板はこの規則で hole_clearance 206 件、塗り直した板は 0。ベタの面積 表 −56.7・裏 −60.9 mm²
- B-3: スタビの足跡に B.CrtYd（箱・ねじの頭 φ3.85・爪の先 10.95 ＋ 0.25）
- 網の差: 92 網のうち GND のビアだけ（+8 −2。−2 は塗りが変わって 0.077 ずれた 1 本島の 2 本目）
- 検査: 道のり（board_facts の gnd_fill）・シルクとマスクの開口・穴と銅の規則と DRC の壊す検査・裏のコートヤード

Co-Authored-By: Claude Opus 5.5 (1M context) <noreply@anthropic.com>
Routing:
- net GND: vias 893 -> 899
