File: projects/cckb-click/pcb/cckb-click_main.kicad_pcb (KiCad board)
At the start: 2 copper layers, 291.2 x 100.7 mm, 185 parts, among them SW1 SKRAAWE010, SW10 SKRAAWE010, SW11 SKRAAWE010, SW12 SKRAAWE010, SW13 SKRAAWE010, SW14 SKRAAWE010, SW15 SKRAAWE010, SW16 SKRAAWE010, SW17 SKRAAWE010, SW18 SKRAAWE010, SW19 SKRAAWE010, SW2 SKRAAWE010, SW20 SKRAAWE010, SW21 SKRAAWE010, SW22 SKRAAWE010, SW23 SKRAAWE010, SW24 SKRAAWE010, SW25 SKRAAWE010, SW26 SKRAAWE010, SW27 SKRAAWE010, SW28 SKRAAWE010, SW29 SKRAAWE010, SW3 SKRAAWE010, SW30 SKRAAWE010, SW31 SKRAAWE010, SW32 SKRAAWE010, SW33 SKRAAWE010, SW34 SKRAAWE010, SW35 SKRAAWE010, SW36 SKRAAWE010, SW37 SKRAAWE010, SW38 SKRAAWE010, SW39 SKRAAWE010, SW4 SKRAAWE010, SW40 SKRAAWE010, SW41 SKRAAWE010, SW42 SKRAAWE010, SW43 SKRAAWE010, SW44 SKRAAWE010, SW45 SKRAAWE010, SW46 SKRAAWE010, SW47 SKRAAWE010, SW48 SKRAAWE010, SW49 SKRAAWE010, SW5 SKRAAWE010, SW50 SKRAAWE010, SW51 SKRAAWE010, SW52 SKRAAWE010, SW53 SKRAAWE010, SW54 SKRAAWE010, SW55 SKRAAWE010, SW56 SKRAAWE010, SW57 SKRAAWE010, SW58 SKRAAWE010, SW59 SKRAAWE010, SW6 SKRAAWE010, SW60 SKRAAWE010, SW61 SKRAAWE010, SW62 SKRAAWE010, SW7 SKRAAWE010, SW8 SKRAAWE010, SW9 SKRAAWE010, U1 SN74LVC595APWR, U2 SN74LVC595APWR

Commit message: cckb-click: 1 回目の監査の直し（基板を配線し直した・枠・ねじの試し刷り・ファーム・検査）
基板（DRC 違反 0・未配線 0・警告 0。sha256 4dc68901…）
- 電池は止めに当たる所に座る（クリップの原点から 0.51 奥）。表の銅を置かない範囲を奥へ広げた: 缶の縁から銅まで 0 → 0.72
- 載せないコンデンサのランド 2 つ（C_BAT = VBAT_SW–GND・C_3V3 = V3V3–GND。1206 と 0805 が載る・JLC は実装しない・ペースト無し）
- 手前の継ぎ目の両側に予備のねじ穴 2 つ。外周のねじ穴を 0.1 外へ（穴の縁から基板の縁まで 1.0）
- パスコンの GND から 595 の GND までを GND の線で引く（31.6 → 22.3 mm）・595 の本体の下の帯に線を通さずビアを先に打つ
  （表の GND のいちばん遠い所 17.2 → 13.3 mm）・電池電圧の線を行の線から 1.8 離す・C_3V3 への線を決まった形で
- 試験用のランドのシルクの輪・ランドの中のビアの禁止・アンテナの禁止域の手前の細い帯を塗らない・DRC の下限をビア φ0.6・穴 0.3 に

枠
- ねじの所の厚い壁を ±2.0 に（下穴のまわりの肉 0.49 → 0.71。幅の広いキーの脇の 3 本は 0.49 のまま）・予備のねじの下穴
- 電源スイッチと XIAO の逃げをパッドの外接 ＋ 0.4 に・指の切り欠きの奥行き 4.5
- ねじの試し刷り coupon_screw_plate（本番の枠から切り出した壁 2 つ ＋ 厚さ 1.6 の当て板。3 番だけ壁を 0.5 厚くした）

ファーム: SPI の MISO（D9・基板では空き）にプルダウン（ボードの pinctrl の写しと突き合わせ）

検査（どれも壊すと落ちる）: 電池の縁から表の銅まで・シルクの図形とマスクの開口・戻りの道のり・電池電圧の線と行の線・
ランドが 0805 と 1206 の標準の足跡を含む・電池クリップの向き（CPL・JLC の部品データの外形）・電池電圧の式・ねじの肉 22 か所・
枠とパッドの隙・ねじの試し刷りが本番の枠と同じ形。全検査 655 passed。

Co-Authored-By: Claude Opus 5.5 (1M context) <noreply@anthropic.com>
Parts:
- added C_3V3: cap_land_unpopulated, C_1206_0805_Land, F.Cu at (53.1, 121.5)
- added C_BAT: cap_land_unpopulated, C_1206_0805_Land, F.Cu at (287.2, 133.0)
- added H28: Hole_M2_2.2, Hole_M2_2.2, F.Cu at (148.3, 148.2)
- added H29: Hole_M2_2.2, Hole_M2_2.2, F.Cu at (161.3, 148.2)
- moved H18 0.10 mm to (293.5, 77.2)
- moved H19 0.10 mm to (293.5, 119.0)
- moved H0 0.10 mm to (16.6, 51.8)
- moved H1 0.10 mm to (54.8, 51.8)
- moved H2 0.10 mm to (92.8, 51.8)
- moved H3 0.10 mm to (130.9, 51.8)
- moved H4 0.10 mm to (150.0, 51.8)
- moved H5 0.10 mm to (169.1, 51.8)
- moved H6 0.10 mm to (207.2, 51.8)
- moved H7 0.10 mm to (245.2, 51.8)
- moved H8 0.10 mm to (283.4, 51.8)
- moved H16 0.10 mm to (6.53, 77.2)
- moved H17 0.10 mm to (6.53, 115.2)
- moved H10 0.10 mm to (104.8, 148.2)
- moved H11 0.10 mm to (140.5, 148.2)
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Routing:
- net GND: track 19.4 -> 64.5 mm, vias 804 -> 810
- net V3V3: track 66.7 -> 80.6 mm, vias 2 -> 5
- net VBAT_SW: track 297.9 -> 305.9 mm, vias 3 -> 2
- net CS: track 27.4 -> 30.8 mm, vias 2 -> 4
- net VBAT_SENSE: track 27.5 -> 30.1 mm
- net U1_U2: track 16.1 -> 18.5 mm
- net SPI_SCK: track 31.7 -> 33.6 mm, vias 2 -> 3
- net SPI_MOSI: track 27.5 -> 28.1 mm

Commit message: cckb-click: 電源スイッチを基板の縁から 2.5 内側へ・つまみの切り欠き・差し込み式の電池の蓋・蓋のねじ穴・角の試し刷り
利用者の決定（2026-10-04）:
- 電源スイッチ MSK12C02 を 1.75 内側へ（本体は縁から 2.50 = JLC の規約・つまみの先は枠の外面の 1.35 内側）。
  枠の右の壁を幅 10・上まで切り欠き、内側は屋根を厚くして塞ぐ。入の向きと印は同じ
- 電池の蓋（cover_battery.stl）: L 字・手前から滑らせる・枠のひさしと溝だけで留まる・無くても使える
- 蓋のねじ穴 H30・H31（非めっき φ2.2・使わない）。電池クリップのコートヤードの口の側の両脇を欠いた
- 角の試し刷り（coupon_corner_plate.stl）: 本番の枠の右手前の角 ＋ 当て板 ＋ つまみ・電池の代わり ＋ 蓋

基板: C_BAT を 1.0 左へ。電池の＋（VBAT_IN）を決まった形に。SPI・595 どうし・電源の枝は、監査した板（4dc68901…）で
Freerouting が引いた線を pcb/freerouted.json から置き直す（引くたびに形が変わらない）。右手前の角の外で前の板と違うのは
VBAT_SW の長い線の右の端だけ。DRC 違反 0・未配線 0・警告 0。板 fe90b1e6…

検査（それぞれ壊すと落ちる）: 本体と縁 2.5・つまみが枠の内側・爪の入る場所・蓋が当たらず滑って抜けて留まる・
蓋のねじ穴と裏の銅・置き直した線が記録と同じ・角の試し刷りが本番の枠と同じ。全検査 677 passed。

Co-Authored-By: Claude Opus 5.5 (1M context) <noreply@anthropic.com>
Parts:
- added H30: Hole_M2_2.2, Hole_M2_2.2, F.Cu at (265.0, 148.2)
- added H31: Hole_M2_2.2, Hole_M2_2.2, F.Cu at (279.0, 148.2)
- moved SW_PWR 1.75 mm to (291.1, 138.1)
- moved C_BAT 1.00 mm to (286.2, 133.0)
Routing:
- net VBAT_SW: track 305.9 -> 303.4 mm
- net VBAT_IN: track 40.5 -> 42.4 mm
- net GND: vias 810 -> 811

Commit message: cckb-click: 試し刷り v2 の結果を本番へ（電源スイッチを 0.75 外へ・切り欠きを利用者が触った形に・下穴 φ1.6・蓋を刷る物から外す）
利用者が試し刷り v2 を刷って決めた（2026-10-04）:
- 電源スイッチ: (ii) 0.75 外。本体は基板の縁から 1.75・つまみの先は基板の縁の 0.30 内・枠の外面の 0.60 内。
  JLC の実装の規約「本体と縁は 2.5 mm 以上」は満たさない（規約より使いやすさ）
- 基板: SW_PWR だけ動かし、角だけ引き直した。角の外の違いは VBAT_SW の長い線の右の端 0.75 だけ。
  DRC 違反 0・未配線 0・警告 0。板 b442b865…。入の向き（端子の網）は同じ
- 枠: 切り欠きは外面へ片側 2.4 広がり、内側の上の縁を 2.0 斜めに（PSW_NOTCH）。入の印は斜面のすぐ内の平らな上面へ。
  下穴 φ1.6（22 個とも。薄い壁も補正しない: 線で 1.50 = 利用者が締めた切れ端と同じ）
- 電池の蓋: 4 つとも使えなかった。刷る物・組んだ絵から外した（枠の口のまわりの形と基板の穴 H30・H31 は前のまま）
- 検査: 「本体が縁から 2.5 以上」を、決めた決まり（つまみの先が縁の 0.30 以上内側・枠から出ない・本体 1.75 を記録）に置き換えた。
  最初の位置・0.1 外・前の位置で落ちる。下穴の径・指先の球・切り欠きの縁の強さ（断面を立体から測る）を足した
- 道具: 本番の枠の下穴 22 個を G-code で測る（tools/slice_main.py）
- 試し刷り v2 は、刷った物と同じ形を出し続ける（位置を本番から測り直した）

Co-Authored-By: Claude Opus 5.5 (1M context) <noreply@anthropic.com>
Parts:
- moved SW_PWR 0.75 mm to (291.9, 138.1)
Routing:
- net VBAT_SW: track 303.4 -> 304.9 mm
- net VBAT_IN: track 42.4 -> 43.1 mm
- net GND: vias 811 -> 812
